File: Battery_Switchover_24V/Battery_Switchover_24V.kicad_pcb (KiCad board)
At the start: 2 copper layers, 188.9 x 89 mm, 164 parts, among them J1 USB_C_Receptacle_USB2.0_14P, J10 ATX_2X3, J11 ATX_2X3, J12 ATX_2X3, J13 ATX_2X3, J2 M8, J4 M8, J5 M8, J6 Conn_01x08, J8 ATX_2X3, J9 ATX_2X3, M1 Fan, Q1 PZT2222AT1G, Q2 PJD50N10AL_L2, Q3 PJD50N10AL_L2, Q4 FDBL86066-F085, Q5 FDBL86066-F085, Q6 FDBL86066-F085, Q7 FDBL86066-F085, SW1 SW_Push, U1 LM25117PSQE_NOPB, U10 LPC11U67JBD48, U11 LM60CIM3, U12 L5973D, U13 AMS1117-3.3, U14 OPA2197xD, U16 LM74610QDGKRQ1, U2 ACS71240LLCBTR-010B3, U3 LPC11U14FBD48-201, U4 ACS71240LLCBTR-010B3, U5 ACS71240LLCBTR-010B3, U6 LM74610QDGKRQ1, U7 ACS71240LLCBTR-010B3, U8 ADS7830IPWR, U9 LMV321, Y1 12.000MHz

Commit message: Added load switches
Parts:
- removed CR1, CR2: PESD5V0S1BL, footprints:SOD882_NXP
- added C63: 10nF, Capacitor_SMD:C_0603_1608Metric, F.Cu at (248.5, 72.5)
- added D16: LED, LED_SMD:LED_0805_2012Metric_Pad1.15x1.40mm_HandSolder, B.Cu at (246.3, 130.6)
- added D17: SM712_SOT23, Package_TO_SOT_SMD:SOT-23, F.Cu at (108.3, 45.6)
- added DS1: OLED_128X64_1.3_I2C, LCD_OLED_I2C:LCD_OLED_128X64_1.3_I2C, B.Cu at (193.8, 87.3)
- added J7: Conn_01x05, Connector_PinHeader_2.54mm:PinHeader_1x05_P2.54mm_Vertical, F.Cu at (234.9, 78.1)
- added Q10: FDBL86066-F085, Package_TO_SOT_SMD:Infineon_PG-HSOF-8-1_ThermalVias, F.Cu at (136.4, 101.0)
- added Q8: FDBL86066-F085, Package_TO_SOT_SMD:Infineon_PG-HSOF-8-1_ThermalVias, F.Cu at (136.4, 77.6)
- added Q9: FDBL86066-F085, Package_TO_SOT_SMD:Infineon_PG-HSOF-8-1_ThermalVias, F.Cu at (136.4, 89.3)
- added R47: 4K7, Resistor_SMD:R_0603_1608Metric, F.Cu at (231.0, 137.5)
- added U15: IRS21867S, Package_SO:SOIC-8_3.9x4.9mm_P1.27mm, F.Cu at (148.0, 81.7)
- added U17: IRS21867S, Package_SO:SOIC-8_3.9x4.9mm_P1.27mm, F.Cu at (148.0, 88.3)
- J1: footprint Connector_USB:USB_C_Receptacle_G-Switch_GT-USB-7051x -> USB_C_Vertical:GCT_USB4145-03-0170-C_REVA2; moved to B.Cu
- R11, R12, R13: moved to F.Cu
- SW1: moved to B.Cu
- U3: value LPC11U14FBD48-201 -> IRS21867S; footprint Package_QFP:LQFP-48_7x7mm_P0.5mm -> Package_SO:SOIC-8_3.9x4.9mm_P1.27mm
- XMER1, XMER2: value CM5441Z101B-10 -> CMX1616; footprint Inductor_THT:Choke_Schaffner_RN116-04-22.5x21.5mm -> CMX1616Z_Choke:FIL_CMX1616Z171B-10; moved to B.Cu
- moved C5 209.4 mm to (240.9, 72.2)
- moved C7 209.4 mm to (242.9, 72.2)
- moved R21 196.6 mm to (218.1, 80.3)
- moved R22 196.6 mm to (218.1, 82.8)
- moved Y1 193.0 mm to (238.9, 87.8)
- moved C57 183.3 mm to (147.6, 139.9)
- moved C59 183.3 mm to (147.6, 151.9)
- moved C13 183.0 mm to (147.0, 127.3)
- moved C6 181.6 mm to (247.7, 90.2)
- moved C4 181.6 mm to (247.7, 87.9)
- moved D2 180.4 mm to (256.6, 71.9)
- moved D4 180.4 mm to (253.6, 71.9)
- moved D5 180.4 mm to (250.6, 71.9)
- moved R11 180.4 mm to (256.1, 76.9), turned to -90 degrees
- moved R12 180.4 mm to (253.6, 76.9), turned to -90 degrees
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Connections:
- C2 pad 2: Net-(C2-Pad2) -> Net-(U10-XTALOUT)
- C3 pad 2: Net-(C3-Pad2) -> Net-(U10-XTALIN)
- D1 pad 3: Net-(D1-K-Pad3) -> USB_D+
- D1 pad 4: Net-(D1-K-Pad4) -> USB_D-
- J10 pad 4: VOUT -> Net-(J10-Pin_4)
- J10 pad 5: VOUT -> Net-(J10-Pin_4)
- J10 pad 6: VOUT -> Net-(J10-Pin_4)
- J11 pad 4: VOUT -> Net-(J10-Pin_4)
- J11 pad 5: VOUT -> Net-(J10-Pin_4)
- J11 pad 6: VOUT -> Net-(J10-Pin_4)
- J12 pad 4: VOUT -> Net-(J12-Pin_4)
- J12 pad 5: VOUT -> Net-(J12-Pin_4)
- J12 pad 6: VOUT -> Net-(J12-Pin_4)
- J13 pad 4: VOUT -> Net-(J12-Pin_4)
- J13 pad 5: VOUT -> Net-(J12-Pin_4)
- J13 pad 6: VOUT -> Net-(J12-Pin_4)
- J8 pad 4: VOUT -> Net-(J8-Pin_4)
- J8 pad 5: VOUT -> Net-(J8-Pin_4)
- J8 pad 6: VOUT -> Net-(J8-Pin_4)
- J9 pad 4: VOUT -> Net-(J8-Pin_4)
- J9 pad 5: VOUT -> Net-(J8-Pin_4)
- J9 pad 6: VOUT -> Net-(J8-Pin_4)
- R3 pad 2: Net-(D1-K-Pad4) -> USB_D-
- R4 pad 2: Net-(D1-K-Pad3) -> USB_D+
- U10 pad 19: unconnected-(U10-USB_DM-Pad19) -> USB_D-
- U10 pad 20: unconnected-(U10-USB_DP-Pad20) -> USB_D+
- U10 pad 28: unconnected-(U10-PIO0_10/SWCLK-Pad28) -> SWCLK
- U10 pad 34: unconnected-(U10-VREFP-Pad34) -> +3.3V
- U10 pad 35: unconnected-(U10-VREFN-Pad35) -> GND
- U10 pad 37: unconnected-(U10-PIO0_15/SWDIO-Pad37) -> SWDIO
- U10 pad 6: unconnected-(U10-PIO2_0-Pad6) -> Net-(U10-XTALIN)
- U10 pad 7: unconnected-(U10-PIO2_1-Pad7) -> Net-(U10-XTALOUT)
- U3 pad 1: unconnected-(U3-PIO1_25-Pad1) -> VOUT
- U3 pad 4: unconnected-(U3-PIO0_1-Pad4) -> VOUT_GNDPWR
- Y1 pad 1: Net-(C3-Pad2) -> Net-(U10-XTALIN)
- Y1 pad 2: Net-(C2-Pad2) -> Net-(U10-XTALOUT)
Other:
- board size 188.9 x 89 mm -> 198.6 x 89 mm
- board text added: "(+) (-)"
- board text added: "FUSE"
