File: Battery_Switchover_24V/Battery_Switchover_24V.kicad_pcb (KiCad board)
At the start: 2 copper layers, 198.6 x 89 mm, 173 parts, among them J1 USB_C_Receptacle_USB2.0_14P, J10 ATX_2X3, J11 ATX_2X3, J12 ATX_2X3, J13 ATX_2X3, J2 M8, J4 M8, J5 M8, J6 Conn_01x08, J7 Conn_01x05, J8 ATX_2X3, J9 ATX_2X3, M1 Fan, Q1 PZT2222AT1G, Q10 FDBL86066-F085, Q2 PJD50N10AL_L2, Q3 PJD50N10AL_L2, Q4 FDBL86066-F085, Q5 FDBL86066-F085, Q6 FDBL86066-F085, Q7 FDBL86066-F085, Q8 FDBL86066-F085, Q9 FDBL86066-F085, SW1 SW_Push, U1 LM25117PSQE_NOPB, U10 LPC11U67JBD48, U11 LM60CIM3, U12 L5973D, U13 AMS1117-3.3, U14 OPA2197xD, U15 IRS21867S, U16 LM74610QDGKRQ1, U17 IRS21867S, U2 ACS71240LLCBTR-010B3, U3 IRS21867S, U4 ACS71240LLCBTR-010B3, U5 ACS71240LLCBTR-010B3, U6 LM74610QDGKRQ1, U7 ACS71240LLCBTR-010B3, U8 ADS7830IPWR, U9 LMV321, Y1 12.000MHz

Commit message: adc pins holes
Parts:
- removed C3: 18pF, Capacitor_SMD:C_0402_1005Metric
- removed U11: LM60CIM3, footprints:MF03A
- removed Y1: 12.000MHz, Crystal:Crystal_SMD_TXC_7M-4Pin_3.2x2.5mm
- added D12: D_Schottky, Diode_SMD:D_SOD-323_HandSoldering, F.Cu at (160.8, 51.6)
- added D13: D, Diode_SMD:D_SOD-323_HandSoldering, F.Cu at (160.8, 46.6)
- added H1: MHole_Pad, MountingHole:MountingHole_2.5mm_Pad_Via, F.Cu at (92.2, 156.2)
- added H2: MHole_Pad, MountingHole:MountingHole_2.5mm_Pad_Via, F.Cu at (176.0, 156.0)
- added H3: MHole_Pad, MountingHole:MountingHole_2.5mm_Pad_Via, F.Cu at (92.2, 72.8)
- added H4: MHole_Pad, MountingHole:MountingHole_2.5mm_Pad_Via, F.Cu at (285.0, 72.8)
- added H5: MHole_Pad, MountingHole:MountingHole_2.5mm_Pad_Via, F.Cu at (285.0, 156.2)
- added H6: MHole_Pad, MountingHole:MountingHole_2.5mm_Pad_Via, F.Cu at (172.9, 72.8)
- added R48: 1K, Resistor_SMD:R_0603_1608Metric, F.Cu at (167.1, 135.7)
- added R49: 1K, Resistor_SMD:R_0603_1608Metric, F.Cu at (167.1, 138.2)
- added U18: LM60CIM3_NOPB, SOT95P251X112-3N:SOT95P251X112-3N, F.Cu at (173.1, 134.1)
- C13, C30, C57, C59, C61: footprint Capacitor_THT:CP_Radial_Tantal_D10.5mm_P5.00mm -> Capacitor_SMD:C_Elec_8x10.2
- C2: value 18pF -> 100nF; footprint Capacitor_SMD:C_0402_1005Metric -> Capacitor_SMD:C_0603_1608Metric
- moved C17 138.9 mm to (311.5, 72.8)
- moved C18 138.9 mm to (311.5, 75.3)
- moved R35 138.9 mm to (319.5, 72.8)
- moved R40 138.9 mm to (319.5, 85.3)
- moved C2 130.5 mm to (167.1, 133.2), turned to 0 degrees
- moved R41 117.7 mm to (314.4, 52.9)
- moved R42 117.7 mm to (314.4, 55.4)
- moved R43 117.7 mm to (314.4, 57.9)
- moved R28 117.7 mm to (302.3, 65.5)
- moved R29 117.7 mm to (306.3, 52.9)
- moved R30 117.7 mm to (306.3, 55.4)
- moved R31 117.7 mm to (306.3, 57.9)
- moved R32 117.7 mm to (306.3, 60.4)
- moved R33 117.7 mm to (306.3, 62.9)
- moved R34 117.7 mm to (306.3, 65.5)
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Connections:
- net Net-(D12-A) renamed VBUS
- C2 pad 1: GND -> +3.3V
- C2 pad 2: Net-(U10-XTALOUT) -> GND
- C29 pad 2: Net-(U1-SW) -> Net-(Q2-S)
- C44 pad 1: +5V -> +3.3V
- C45 pad 1: +5V -> +3.3V
- J7 pad 2: unconnected-(J7-Pin_2-Pad2) -> RESET
- J7 pad 3: SWCLK -> UART0_RX
- J7 pad 4: SWDIO -> UART0_TX
- L2 pad 1: Net-(U1-SW) -> Net-(Q2-S)
- Q2 pad 1: (no net) -> Net-(Q2-G)
- Q2 pad 2: (no net) -> VIN
- Q2 pad 3: (no net) -> Net-(Q2-S)
- Q3 pad 1: (no net) -> Net-(Q3-G)
- Q3 pad 2: (no net) -> Net-(Q2-S)
- Q3 pad 3: (no net) -> GND
- U1 pad 15: Net-(U1-LO) -> Net-(Q3-G)
- U1 pad 17: Net-(U1-SW) -> Net-(Q2-S)
- U1 pad 18: Net-(U1-HO) -> Net-(Q2-G)
- U10 pad 12: unconnected-(U10-PIO2_2-Pad12) -> LOAD3_EN
- U10 pad 13: unconnected-(U10-PIO1_20-Pad13) -> Battery_Status_LED
- U10 pad 14: unconnected-(U10-PIO0_3-Pad14) -> Net-(U10-PIO0_3)
- U10 pad 15: unconnected-(U10-PIO0_4-Pad15) -> SCL
- U10 pad 16: unconnected-(U10-PIO0_5-Pad16) -> SDA
- U10 pad 18: unconnected-(U10-PIO1_23-Pad18) -> FAN_CONTROL
- U10 pad 25: unconnected-(U10-PIO1_21-Pad25) -> Fan_Status_LED
- U10 pad 28: SWCLK -> unconnected-(U10-PIO0_10/SWCLK-Pad28)
- U10 pad 29: unconnected-(U10-PIO0_22-Pad29) -> VIOUT2
- U10 pad 3: unconnected-(U10-PIO0_0-Pad3) -> RESET
- U10 pad 30: unconnected-(U10-PIO0_11-Pad30) -> BATT_CURRENT
- U10 pad 31: unconnected-(U10-PIO0_12-Pad31) -> BOARD_TEMPERATURE
- U10 pad 32: unconnected-(U10-PIO0_13-Pad32) -> ADC_VBatt
- U10 pad 33: unconnected-(U10-PIO0_14-Pad33) -> ADC_VIN
- U10 pad 36: unconnected-(U10-PIO1_13-Pad36) -> Main_Voltage_LED
- U10 pad 37: SWDIO -> unconnected-(U10-PIO0_15/SWDIO-Pad37)
- U10 pad 38: unconnected-(U10-PIO0_16-Pad38) -> VIOUT1
- U10 pad 39: unconnected-(U10-PIO0_23-Pad39) -> VIOUT3
- U10 pad 4: unconnected-(U10-PIO0_1-Pad4) -> BATTERY_OW_TEMP
- U10 pad 45: unconnected-(U10-PIO0_18-Pad45) -> UART0_RX
- U10 pad 46: unconnected-(U10-PIO0_19-Pad46) -> UART0_TX
- U10 pad 6: Net-(U10-XTALIN) -> LOAD1_EN
- U10 pad 7: Net-(U10-XTALOUT) -> LOAD2_EN
- U14 pad 1: ADC_Batt -> ADC_VBatt
- U14 pad 2: ADC_Batt -> ADC_VBatt
- U14 pad 6: ADC_In -> ADC_VIN
- U14 pad 7: ADC_In -> ADC_VIN
- U14 pad 8: +5V -> +3.3V
Routing:
- net Net-(D6-A1): track 0.00 -> 51.5 mm
- net Net-(D16-A): track 0.00 -> 51.5 mm
- net Net-(D16-K): track 0.00 -> 33.0 mm
- added copper zone on In1.Cu, net GND
Other:
- copper layers 2 -> 4

Commit message: load switches positioned
Parts:
- removed C10: 100pF, Capacitor_SMD:C_1206_3216Metric
- removed C11, C54, C55: 1nF, Capacitor_SMD:C_1206_3216Metric
- removed C13: 330uF, Capacitor_SMD:C_Elec_8x10.2
- removed D7: P6SMBJ26A, Diode_SMD:D_SMB_Handsoldering
- removed XMER2: CMX1616, CMX1616Z_Choke:FIL_CMX1616Z171B-10
- added BZ1: Buzzer, Buzzer_Beeper:MagneticBuzzer_CUI_CMT-8504-100-SMT, B.Cu at (239.3, 51.1)
- added C3: 10nF, Capacitor_SMD:C_0603_1608Metric, F.Cu at (231.7, 34.7)
- added C64: 10nF, Capacitor_SMD:C_0603_1608Metric, F.Cu at (231.7, 37.2)
- added D18: P6SMBJ26A, Diode_SMD:D_SMB_Handsoldering, F.Cu at (125.4, 103.6)
- added D19: P6SMBJ26A, Diode_SMD:D_SMB_Handsoldering, F.Cu at (125.7, 78.2)
- added D20: P6SMBJ26A, Diode_SMD:D_SMB_Handsoldering, F.Cu at (125.4, 128.3)
- added Q11: BC817, Package_TO_SOT_SMD:SOT-23, F.Cu at (246.5, 35.8)
- added R50: 1K, Resistor_SMD:R_0603_1608Metric, F.Cu at (231.7, 39.7)
- added R51: 1K, Resistor_SMD:R_0603_1608Metric, F.Cu at (231.7, 42.2)
- added R52: 1K, Resistor_SMD:R_0603_1608Metric, F.Cu at (231.7, 44.7)
- added SW2: SW_Push, Button_Switch_SMD:SW_SPST_TL3305A, B.Cu at (238.9, 36.5)
- added SW3: SW_Push, Button_Switch_SMD:SW_SPST_TL3305A, B.Cu at (238.9, 42.5)
- C31: moved to F.Cu
- moved R3 237.1 mm to (280.4, 25.3)
- moved R4 237.1 mm to (278.2, 25.3)
- moved R1 228.1 mm to (276.4, 25.1)
- moved C31 180.0 mm to (172.1, 118.5)
- moved C2 167.3 mm to (294.4, 24.6)
- moved R48 149.8 mm to (270.6, 27.4)
- moved R49 149.8 mm to (270.6, 29.9)
- moved U13 138.5 mm to (386.8, 69.9)
- moved C16 136.8 mm to (190.8, 116.3)
- moved C52 135.7 mm to (184.6, 115.8)
- moved C53 130.6 mm to (184.6, 112.9)
- moved C14 130.2 mm to (168.8, 95.8)
- moved R26 124.2 mm to (194.7, 114.4)
- moved R25 120.8 mm to (196.1, 108.8)
- moved R27 119.5 mm to (194.7, 112.0)
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Connections:
- C56 pad 2: VOUT_GNDPWR -> GND
- C57 pad 2: VOUT_GNDPWR -> GND
- C58 pad 2: VOUT_GNDPWR -> GND
- C59 pad 2: VOUT_GNDPWR -> GND
- C60 pad 2: VOUT_GNDPWR -> GND
- C61 pad 2: VOUT_GNDPWR -> GND
- D14 pad 1: VOUT_GNDPWR -> GND
- J10 pad 4: Net-(J10-Pin_4) -> Net-(D18-A2)
- J10 pad 5: Net-(J10-Pin_4) -> Net-(D18-A2)
- J10 pad 6: Net-(J10-Pin_4) -> Net-(D18-A2)
- J11 pad 4: Net-(J10-Pin_4) -> Net-(D18-A2)
- J11 pad 5: Net-(J10-Pin_4) -> Net-(D18-A2)
- J11 pad 6: Net-(J10-Pin_4) -> Net-(D18-A2)
- J12 pad 4: Net-(J12-Pin_4) -> Net-(D20-A2)
- J12 pad 5: Net-(J12-Pin_4) -> Net-(D20-A2)
- J12 pad 6: Net-(J12-Pin_4) -> Net-(D20-A2)
- J13 pad 4: Net-(J12-Pin_4) -> Net-(D20-A2)
- J13 pad 5: Net-(J12-Pin_4) -> Net-(D20-A2)
- J13 pad 6: Net-(J12-Pin_4) -> Net-(D20-A2)
- J8 pad 4: Net-(J8-Pin_4) -> Net-(D19-A2)
- J8 pad 5: Net-(J8-Pin_4) -> Net-(D19-A2)
- J8 pad 6: Net-(J8-Pin_4) -> Net-(D19-A2)
- J9 pad 4: Net-(J8-Pin_4) -> Net-(D19-A2)
- J9 pad 5: Net-(J8-Pin_4) -> Net-(D19-A2)
- J9 pad 6: Net-(J8-Pin_4) -> Net-(D19-A2)
- Q10 pad 1: (no net) -> unconnected-(Q10-G-Pad1)
- Q10 pad 2: (no net) -> Net-(D20-A2)
- Q10 pad 3: (no net) -> VOUT
- Q4 pad 1: (no net) -> Net-(Q4-G)
- Q4 pad 2: (no net) -> VBATT
- Q4 pad 3: (no net) -> VOUT
- Q5 pad 1: (no net) -> Net-(Q4-G)
- Q5 pad 2: (no net) -> VBATT
- Q5 pad 3: (no net) -> VOUT
- Q6 pad 1: (no net) -> Net-(Q6-G)
- Q6 pad 2: (no net) -> VIN
- Q6 pad 3: (no net) -> VOUT
- Q7 pad 1: (no net) -> Net-(Q6-G)
- Q7 pad 2: (no net) -> VIN
- Q7 pad 3: (no net) -> VOUT
- Q8 pad 1: (no net) -> unconnected-(Q8-G-Pad1)
- Q8 pad 2: (no net) -> Net-(D19-A2)
- Q8 pad 3: (no net) -> VOUT
- Q9 pad 1: (no net) -> unconnected-(Q9-G-Pad1)
- Q9 pad 2: (no net) -> Net-(D18-A2)
- Q9 pad 3: (no net) -> VOUT
- U10 pad 10: unconnected-(U10-PIO0_20-Pad10) -> BUTTON1
- U10 pad 17: unconnected-(U10-PIO0_21-Pad17) -> BUTTON2
- U10 pad 42: unconnected-(U10-PIO0_17-Pad42) -> BUZZER
- U15 pad 4: VOUT_GNDPWR -> GND
- U16 pad 2: Net-(U16-GATE_DRIVE) -> Net-(Q6-G)
- U16 pad 6: Net-(U16-GATE_DRIVE) -> Net-(Q6-G)
- U16 pad 8: Net-(D7-A2) -> VOUT
- U17 pad 4: VOUT_GNDPWR -> GND
- U2 pad 3: VOUT_GNDPWR -> GND
- U2 pad 4: VOUT_GNDPWR -> GND
- U3 pad 4: VOUT_GNDPWR -> GND
- U4 pad 3: VOUT_GNDPWR -> GND
- U4 pad 4: VOUT_GNDPWR -> GND
- U5 pad 3: VOUT_GNDPWR -> GND
- U5 pad 4: VOUT_GNDPWR -> GND
- U6 pad 2: Net-(U6-GATE_DRIVE) -> Net-(Q4-G)
- U6 pad 6: Net-(U6-GATE_DRIVE) -> Net-(Q4-G)
- U6 pad 8: Net-(D7-A2) -> VOUT
- XMER1 pad 1: Net-(D16-K) -> Net-(D6-A1)
- XMER1 pad 2: Net-(D6-A1) -> Net-(D16-K)
- XMER1 pad 3: GND -> VIN
- XMER1 pad 4: VIN -> GND
Routing:
- net VOUT: track 0.00 -> 429.7 mm
- net VIN: track 0.00 -> 97.9 mm
- net Net-(D16-K): track 33.0 -> 129.4 mm
- net LOAD3_GND_RETURN: track 0.00 -> 54.0 mm
- net Net-(D19-A2): track 0.00 -> 38.7 mm
- net LOAD1_GND_RETURN: track 0.00 -> 37.5 mm
- net Net-(D18-A2): track 0.00 -> 37.1 mm
- net Net-(D20-A2): track 0.00 -> 37.1 mm
- net Net-(D6-A1): track 51.5 -> 85.6 mm
- net VBATT: track 0.00 -> 30.5 mm
- net LOAD2_GND_RETURN: track 0.00 -> 29.8 mm
- net GND: track 0.00 -> 3.63 mm
- added copper zone on B.Cu, net GND
- added copper zone on F.Cu, net GND

Commit message: board placement
Parts:
- moved U6 60.8 mm to (159.8, 146.7), turned to 180 degrees
- moved C14 45.8 mm to (141.9, 58.7)
- moved C29 45.8 mm to (145.0, 53.8)
- moved C47 45.8 mm to (148.8, 53.7)
- moved C48 45.8 mm to (129.5, 55.0)
- moved C49 45.8 mm to (132.7, 57.6)
- moved C50 45.8 mm to (132.7, 54.9)
- moved C51 45.8 mm to (125.8, 59.0)
- moved D13 45.8 mm to (145.6, 49.9)
- moved R14 45.8 mm to (135.5, 47.9)
- moved R15 45.8 mm to (132.1, 49.8)
- moved R16 45.8 mm to (132.0, 51.7)
- moved R23 45.8 mm to (129.5, 57.6)
- moved R24 45.8 mm to (145.1, 51.8)
- moved U1 45.8 mm to (138.8, 52.8)
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Routing:
- net VIN: track 97.9 -> 59.8 mm
- net VOUT: track 429.7 -> 394.2 mm
- net Net-(D18-A2): track 37.1 -> 27.9 mm
- net Net-(D20-A2): track 37.1 -> 28.4 mm
- net Net-(D19-A2): track 38.7 -> 31.2 mm
- net LOAD3_GND_RETURN: track 54.0 -> 47.9 mm
- net LOAD1_GND_RETURN: track 37.5 -> 31.7 mm
- net GND: track 3.63 -> 0.00 mm
- net LOAD2_GND_RETURN: track 29.8 -> 30.6 mm
- added copper zone on F.Cu, net LOAD1_GND_RETURN
- added copper zone on F.Cu, net LOAD2_GND_RETURN
- added copper zone on F.Cu, net LOAD3_GND_RETURN
- added copper zone on B.Cu, net Net-(D16-K)
- added copper zone on F.Cu, net Net-(D16-K)
- added copper zone on F.Cu, net Net-(D18-A2)
- added copper zone on F.Cu, net Net-(D19-A2)
- added copper zone on F.Cu, net Net-(D20-A2)
- added copper zone on B.Cu, net Net-(D6-A1)
- added copper zone on F.Cu, net Net-(D6-A1)
- added copper zone on F.Cu, net VBATT
- added copper zone on F.Cu, net VIN
- added copper zone on B.Cu, net VOUT
- added copper zone on F.Cu, net VOUT
- removed copper zone on F.Cu, net GND
